File: V2/1800122-V2.kicad_pcb (KiCad board)
At the start: 2 copper layers, 0 parts

Commit message: Added updated KiCAD files with local repos
Parts:
- added C1: 15p, Capacitor_SMD:C_0402_1005Metric_Pad0.74x0.62mm_HandSolder, F.Cu at (-33.1, 117.0)
- added C2: 15p, Capacitor_SMD:C_0402_1005Metric_Pad0.74x0.62mm_HandSolder, F.Cu at (-33.1, 119.0)
- added C3: 10u, Capacitor_SMD:C_0402_1005Metric_Pad0.74x0.62mm_HandSolder, F.Cu at (-33.1, 120.9)
- added C4: 100n, Capacitor_SMD:C_0402_1005Metric_Pad0.74x0.62mm_HandSolder, F.Cu at (-33.1, 122.9)
- added C5: 10u, Capacitor_SMD:C_0402_1005Metric_Pad0.74x0.62mm_HandSolder, F.Cu at (-33.1, 124.9)
- added D_1: D, Diode_SMD:D_SOD-123, B.Cu at (44.5, 47.1)
- added D_10: D, Diode_SMD:D_SOD-123, B.Cu at (249.2, 47.1)
- added D_100: D, Diode_SMD:D_SOD-123, B.Cu at (44.5, 151.9)
- added D_101: D, Diode_SMD:D_SOD-123, B.Cu at (63.5, 151.9)
- added D_102: D, Diode_SMD:D_SOD-123, B.Cu at (82.5, 151.9)
- added D_103: D, Diode_SMD:D_SOD-123, B.Cu at (101.6, 161.4)
- added D_104: D, Diode_SMD:D_SOD-123, B.Cu at (137.3, 151.9)
- added D_105: D, Diode_SMD:D_SOD-123, B.Cu at (168.3, 151.9)
- added D_106: D, Diode_SMD:D_SOD-123, B.Cu at (187.3, 151.9)
- added D_107: D, Diode_SMD:D_SOD-123, B.Cu at (206.4, 151.9)
- added D_108: D, Diode_SMD:D_SOD-123, B.Cu at (225.4, 151.9)
- added D_109: D, Diode_SMD:D_SOD-123, B.Cu at (244.5, 151.9)
- added D_11: D, Diode_SMD:D_SOD-123, B.Cu at (268.3, 47.1)
- added D_110: D, Diode_SMD:D_SOD-123, B.Cu at (263.5, 151.9)
- added D_111: D, Diode_SMD:D_SOD-123, B.Cu at (282.6, 151.9)
- added D_112: D, Diode_SMD:D_SOD-123, B.Cu at (301.6, 151.9)
- added D_113: D, Diode_SMD:D_SOD-123, B.Cu at (320.7, 151.9)
- added D_114: D, Diode_SMD:D_SOD-123, B.Cu at (339.7, 151.9)
- added D_115: D, Diode_SMD:D_SOD-123, B.Cu at (370.7, 151.9)
- added D_116: D, Diode_SMD:D_SOD-123, B.Cu at (406.4, 156.6)
- added D_117: D, Diode_SMD:D_SOD-123, B.Cu at (54.0, 170.9)
- added D_118: D, Diode_SMD:D_SOD-123, B.Cu at (82.5, 170.9)
- added D_119: D, Diode_SMD:D_SOD-123, B.Cu at (127.8, 170.9)
- added D_12: D, Diode_SMD:D_SOD-123, B.Cu at (287.3, 47.1)
- added D_120: D, Diode_SMD:D_SOD-123, B.Cu at (151.6, 170.9)
- added D_121: D, Diode_SMD:D_SOD-123, B.Cu at (175.4, 170.9)
- added D_122: D, Diode_SMD:D_SOD-123, B.Cu at (196.8, 170.9)
- added D_123: D, Diode_SMD:D_SOD-123, B.Cu at (265.9, 170.9)
- added D_124: D, Diode_SMD:D_SOD-123, B.Cu at (337.3, 170.9)
- added D_125: D, Diode_SMD:D_SOD-123, B.Cu at (361.2, 170.9)
- added D_126: D, Diode_SMD:D_SOD-123, B.Cu at (387.4, 175.7)
- added D_127: D, Diode_SMD:D_SOD-123, B.Cu at (406.4, 175.7)
- added D_128: D, Diode_SMD:D_SOD-123, B.Cu at (425.4, 175.7)
- added D_13: D, Diode_SMD:D_SOD-123, B.Cu at (306.4, 47.1)
- added D_14: D, Diode_SMD:D_SOD-123, B.Cu at (339.7, 47.1)
- added D_15: D, Diode_SMD:D_SOD-123, B.Cu at (358.8, 47.1)
- added D_16: D, Diode_SMD:D_SOD-123, B.Cu at (377.8, 47.1)
- added D_17: D, Diode_SMD:D_SOD-123, B.Cu at (396.9, 47.1)
- added D_18: D, Diode_SMD:D_SOD-123, B.Cu at (415.9, 47.1)
- added D_19: D, Diode_SMD:D_SOD-123, B.Cu at (435.0, 47.1)
- added D_2: D, Diode_SMD:D_SOD-123, B.Cu at (82.5, 47.1)
- added D_20: D, Diode_SMD:D_SOD-123, B.Cu at (82.5, 66.2)
- added D_21: D, Diode_SMD:D_SOD-123, B.Cu at (101.6, 66.2)
- added D_22: D, Diode_SMD:D_SOD-123, B.Cu at (120.7, 66.2)
- added D_23: D, Diode_SMD:D_SOD-123, B.Cu at (139.7, 66.2)
- added D_24: D, Diode_SMD:D_SOD-123, B.Cu at (158.8, 66.2)
- added D_25: D, Diode_SMD:D_SOD-123, B.Cu at (177.8, 66.2)
- added D_26: D, Diode_SMD:D_SOD-123, B.Cu at (211.1, 66.2)
- added D_27: D, Diode_SMD:D_SOD-123, B.Cu at (230.2, 66.2)
- added D_28: D, Diode_SMD:D_SOD-123, B.Cu at (249.2, 66.2)
- added D_29: D, Diode_SMD:D_SOD-123, B.Cu at (268.3, 66.2)
- added D_3: D, Diode_SMD:D_SOD-123, B.Cu at (101.6, 47.1)
- added D_30: D, Diode_SMD:D_SOD-123, B.Cu at (287.3, 66.2)
- added D_31: D, Diode_SMD:D_SOD-123, B.Cu at (306.4, 66.2)
- added D_32: D, Diode_SMD:D_SOD-123, B.Cu at (339.7, 66.2)
- added D_33: D, Diode_SMD:D_SOD-123, B.Cu at (358.8, 66.2)
- added D_34: D, Diode_SMD:D_SOD-123, B.Cu at (377.8, 66.2)
- added D_35: D, Diode_SMD:D_SOD-123, B.Cu at (396.9, 66.2)
- added D_36: D, Diode_SMD:D_SOD-123, B.Cu at (415.9, 66.2)
- added D_37: D, Diode_SMD:D_SOD-123, B.Cu at (435.0, 66.2)
- added D_38: D, Diode_SMD:D_SOD-123, B.Cu at (44.5, 94.7)
- added D_39: D, Diode_SMD:D_SOD-123, B.Cu at (63.5, 94.7)
- added D_4: D, Diode_SMD:D_SOD-123, B.Cu at (120.7, 47.1)
- added D_40: D, Diode_SMD:D_SOD-123, B.Cu at (82.5, 94.7)
- added D_41: D, Diode_SMD:D_SOD-123, B.Cu at (101.6, 94.7)
- added D_42: D, Diode_SMD:D_SOD-123, B.Cu at (125.4, 94.7)
- added D_43: D, Diode_SMD:D_SOD-123, B.Cu at (144.5, 94.7)
- added D_44: D, Diode_SMD:D_SOD-123, B.Cu at (163.5, 94.7)
- added D_45: D, Diode_SMD:D_SOD-123, B.Cu at (182.6, 94.7)
- added D_46: D, Diode_SMD:D_SOD-123, B.Cu at (201.6, 94.7)
- added D_47: D, Diode_SMD:D_SOD-123, B.Cu at (220.7, 94.7)
- added D_48: D, Diode_SMD:D_SOD-123, B.Cu at (239.7, 94.7)
- added D_49: D, Diode_SMD:D_SOD-123, B.Cu at (258.8, 94.7)
- added D_5: D, Diode_SMD:D_SOD-123, B.Cu at (139.7, 47.1)
- added D_50: D, Diode_SMD:D_SOD-123, B.Cu at (277.8, 94.7)
- added D_51: D, Diode_SMD:D_SOD-123, B.Cu at (296.9, 94.7)
- added D_52: D, Diode_SMD:D_SOD-123, B.Cu at (315.9, 94.7)
- added D_53: D, Diode_SMD:D_SOD-123, B.Cu at (335.0, 94.7)
- added D_54: D, Diode_SMD:D_SOD-123, B.Cu at (354.0, 94.7)
- added D_55: D, Diode_SMD:D_SOD-123, B.Cu at (382.6, 94.7)
- added D_56: D, Diode_SMD:D_SOD-123, B.Cu at (415.9, 94.7)
- added D_57: D, Diode_SMD:D_SOD-123, B.Cu at (435.0, 94.7)
- added D_58: D, Diode_SMD:D_SOD-123, B.Cu at (454.0, 94.7)
- added D_59: D, Diode_SMD:D_SOD-123, B.Cu at (44.5, 113.8)
- added D_6: D, Diode_SMD:D_SOD-123, B.Cu at (158.8, 47.1)
- added D_60: D, Diode_SMD:D_SOD-123, B.Cu at (63.5, 113.8)
- added D_61: D, Diode_SMD:D_SOD-123, B.Cu at (82.5, 113.8)
- added D_62: D, Diode_SMD:D_SOD-123, B.Cu at (101.6, 113.8)
- added D_63: D, Diode_SMD:D_SOD-123, B.Cu at (130.2, 113.8)
- added D_64: D, Diode_SMD:D_SOD-123, B.Cu at (154.0, 113.8)
- added D_65: D, Diode_SMD:D_SOD-123, B.Cu at (173.0, 113.8)
- added D_66: D, Diode_SMD:D_SOD-123, B.Cu at (192.1, 113.8)
- added D_67: D, Diode_SMD:D_SOD-123, B.Cu at (211.1, 113.8)
- added D_68: D, Diode_SMD:D_SOD-123, B.Cu at (230.2, 113.8)
- added D_69: D, Diode_SMD:D_SOD-123, B.Cu at (249.2, 113.8)
- added D_7: D, Diode_SMD:D_SOD-123, B.Cu at (177.8, 47.1)
- added D_70: D, Diode_SMD:D_SOD-123, B.Cu at (268.3, 113.8)
- added D_71: D, Diode_SMD:D_SOD-123, B.Cu at (287.3, 113.8)
- added D_72: D, Diode_SMD:D_SOD-123, B.Cu at (306.4, 113.8)
- added D_73: D, Diode_SMD:D_SOD-123, B.Cu at (325.4, 113.8)
- added D_74: D, Diode_SMD:D_SOD-123, B.Cu at (344.5, 113.8)
- added D_75: D, Diode_SMD:D_SOD-123, B.Cu at (363.5, 113.8)
- added D_76: D, Diode_SMD:D_SOD-123, B.Cu at (387.4, 113.8)
- added D_77: D, Diode_SMD:D_SOD-123, B.Cu at (415.9, 113.8)
- added D_78: D, Diode_SMD:D_SOD-123, B.Cu at (435.0, 113.8)
- added D_79: D, Diode_SMD:D_SOD-123, B.Cu at (454.0, 113.8)
- added D_8: D, Diode_SMD:D_SOD-123, B.Cu at (211.1, 47.1)
- added D_80: D, Diode_SMD:D_SOD-123, B.Cu at (44.5, 132.8)
- added D_81: D, Diode_SMD:D_SOD-123, B.Cu at (63.5, 132.8)
- added D_82: D, Diode_SMD:D_SOD-123, B.Cu at (82.5, 132.8)
- added D_83: D, Diode_SMD:D_SOD-123, B.Cu at (101.6, 132.8)
- added D_84: D, Diode_SMD:D_SOD-123, B.Cu at (132.6, 132.8)
- added D_85: D, Diode_SMD:D_SOD-123, B.Cu at (158.8, 132.8)
- added D_86: D, Diode_SMD:D_SOD-123, B.Cu at (177.8, 132.8)
- added D_87: D, Diode_SMD:D_SOD-123, B.Cu at (196.8, 132.8)
- added D_88: D, Diode_SMD:D_SOD-123, B.Cu at (215.9, 132.8)
- added D_89: D, Diode_SMD:D_SOD-123, B.Cu at (234.9, 132.8)
- added D_9: D, Diode_SMD:D_SOD-123, B.Cu at (230.2, 47.1)
- added D_90: D, Diode_SMD:D_SOD-123, B.Cu at (254.0, 132.8)
- added D_91: D, Diode_SMD:D_SOD-123, B.Cu at (273.1, 132.8)
- added D_92: D, Diode_SMD:D_SOD-123, F.Cu at (-12.7, 147.3)
- added D_93: D, Diode_SMD:D_SOD-123, F.Cu at (-12.7, 150.6)
- added D_94: D, Diode_SMD:D_SOD-123, B.Cu at (330.2, 132.8)
- added D_95: D, Diode_SMD:D_SOD-123, B.Cu at (349.2, 132.8)
- added D_96: D, Diode_SMD:D_SOD-123, B.Cu at (380.2, 132.8)
- added D_97: D, Diode_SMD:D_SOD-123, B.Cu at (415.9, 132.8)
- added D_98: D, Diode_SMD:D_SOD-123, F.Cu at (-6.92, 113.8)
- added D_99: D, Diode_SMD:D_SOD-123, F.Cu at (-6.92, 117.1)
- added J1: USB_C_Receptacle_USB2.0_16P, Connector_USB:USB_C_Receptacle_GCT_USB4105-xx-A_16P_TopMnt_Horizontal, F.Cu at (-50.5, 121.3)
- added J2: Conn_01x03, Connector_JST:JST_SH_SM03B-SRSS-TB_1x03-1MP_P1.00mm_Horizontal, F.Cu at (-45.8, 138.5)
- added K_1: KEYSW, 122-LIB:SW_Hotswap_Kailh_MX_1.00u_PnP, F.Cu at (38.1, 38.1)
- added K_10: KEYSW, 122-LIB:SW_Hotswap_Kailh_MX_1.00u_PnP, F.Cu at (242.9, 38.1)
- added K_100: KEYSW, 122-LIB:SW_Hotswap_Kailh_MX_1.00u_PnP, F.Cu at (38.1, 142.9)
- added K_101: KEYSW, 122-LIB:SW_Hotswap_Kailh_MX_1.00u_PnP, F.Cu at (57.1, 142.9)
- added K_102: KEYSW, 122-LIB:SW_Hotswap_Kailh_MX_1.00u_PnP, F.Cu at (76.2, 142.9)
- added K_103: KEYSW, 122-LIB:SW_Hotswap_Kailh_MX_1.00u_PnP, F.Cu at (95.2, 152.4)
- added K_104: KEYSW, 122-LIB:SW_Hotswap_Kailh_MX_1.00u_PnP, F.Cu at (131.0, 142.9)
- added K_105: KEYSW, 122-LIB:SW_Hotswap_Kailh_MX_1.00u_PnP, F.Cu at (161.9, 142.9)
- added K_106: KEYSW, 122-LIB:SW_Hotswap_Kailh_MX_1.00u_PnP, F.Cu at (181.0, 142.9)
- added K_107: KEYSW, 122-LIB:SW_Hotswap_Kailh_MX_1.00u_PnP, F.Cu at (200.0, 142.9)
- added K_108: KEYSW, 122-LIB:SW_Hotswap_Kailh_MX_1.00u_PnP, F.Cu at (219.1, 142.9)
- added K_109: KEYSW, 122-LIB:SW_Hotswap_Kailh_MX_1.00u_PnP, F.Cu at (238.1, 142.9)
- added K_11: KEYSW, 122-LIB:SW_Hotswap_Kailh_MX_1.00u_PnP, F.Cu at (261.9, 38.1)
- added K_110: KEYSW, 122-LIB:SW_Hotswap_Kailh_MX_1.00u_PnP, F.Cu at (257.2, 142.9)
- added K_111: KEYSW, 122-LIB:SW_Hotswap_Kailh_MX_1.00u_PnP, F.Cu at (276.2, 142.9)
- added K_112: KEYSW, 122-LIB:SW_Hotswap_Kailh_MX_1.00u_PnP, F.Cu at (295.3, 142.9)
- added K_113: KEYSW, 122-LIB:SW_Hotswap_Kailh_MX_1.00u_PnP, F.Cu at (314.3, 142.9)
- added K_114: KEYSW, 122-LIB:SW_Hotswap_Kailh_MX_1.00u_PnP, F.Cu at (333.4, 142.9)
- added K_115: KEYSW, 122-LIB:SW_Hotswap_Kailh_MX_1.00u_PnP, F.Cu at (364.3, 142.9)
- added K_116: KEYSW, 122-LIB:SW_Hotswap_Kailh_MX_1.00u_PnP, F.Cu at (400.1, 147.6)
- added K_117: KEYSW, 122-LIB:SW_Hotswap_Kailh_MX_1.00u_PnP, F.Cu at (47.6, 161.9)
- added K_118: KEYSW, 122-LIB:SW_Hotswap_Kailh_MX_1.00u_PnP, F.Cu at (76.2, 161.9)
- added K_119: KEYSW, 122-LIB:SW_Hotswap_Kailh_MX_1.00u_PnP, F.Cu at (121.4, 161.9)
- added K_12: KEYSW, 122-LIB:SW_Hotswap_Kailh_MX_1.00u_PnP, F.Cu at (281.0, 38.1)
- added K_120: KEYSW, 122-LIB:SW_Hotswap_Kailh_MX_1.00u_PnP, F.Cu at (145.3, 161.9)
- added K_121: KEYSW, 122-LIB:SW_Hotswap_Kailh_MX_1.00u_PnP, F.Cu at (169.1, 161.9)
- added K_122: KEYSW, 122-LIB:SW_Hotswap_Kailh_MX_1.00u_PnP, F.Cu at (190.5, 161.9)
- added K_123: KEYSW, 122-LIB:SW_Hotswap_Kailh_MX_1.00u_PnP, F.Cu at (259.6, 161.9)
- added K_124: KEYSW, 122-LIB:SW_Hotswap_Kailh_MX_1.00u_PnP, F.Cu at (331.0, 161.9)
- added K_125: KEYSW, 122-LIB:SW_Hotswap_Kailh_MX_1.00u_PnP, F.Cu at (354.8, 161.9)
- added K_126: KEYSW, 122-LIB:SW_Hotswap_Kailh_MX_1.00u_PnP, F.Cu at (381.0, 166.7)
- added K_127: KEYSW, 122-LIB:SW_Hotswap_Kailh_MX_1.00u_PnP, F.Cu at (400.1, 166.7)
- added K_128: KEYSW, 122-LIB:SW_Hotswap_Kailh_MX_1.00u_PnP, F.Cu at (419.1, 166.7)
- added K_13: KEYSW, 122-LIB:SW_Hotswap_Kailh_MX_1.00u_PnP, F.Cu at (300.0, 38.1)
- added K_14: KEYSW, 122-LIB:SW_Hotswap_Kailh_MX_1.00u_PnP, F.Cu at (333.4, 38.1)
- added K_15: KEYSW, 122-LIB:SW_Hotswap_Kailh_MX_1.00u_PnP, F.Cu at (352.4, 38.1)
- added K_16: KEYSW, 122-LIB:SW_Hotswap_Kailh_MX_1.00u_PnP, F.Cu at (371.5, 38.1)
- added K_17: KEYSW, 122-LIB:SW_Hotswap_Kailh_MX_1.00u_PnP, F.Cu at (390.5, 38.1)
- added K_18: KEYSW, 122-LIB:SW_Hotswap_Kailh_MX_1.00u_PnP, F.Cu at (409.6, 38.1)
- added K_19: KEYSW, 122-LIB:SW_Hotswap_Kailh_MX_1.00u_PnP, F.Cu at (428.6, 38.1)
- added K_2: KEYSW, 122-LIB:SW_Hotswap_Kailh_MX_1.00u_PnP, F.Cu at (76.2, 38.1)
- added K_20: KEYSW, 122-LIB:SW_Hotswap_Kailh_MX_1.00u_PnP, F.Cu at (76.2, 57.1)
- added K_21: KEYSW, 122-LIB:SW_Hotswap_Kailh_MX_1.00u_PnP, F.Cu at (95.2, 57.1)
- added K_22: KEYSW, 122-LIB:SW_Hotswap_Kailh_MX_1.00u_PnP, F.Cu at (114.3, 57.1)
- added K_23: KEYSW, 122-LIB:SW_Hotswap_Kailh_MX_1.00u_PnP, F.Cu at (133.3, 57.1)
- added K_24: KEYSW, 122-LIB:SW_Hotswap_Kailh_MX_1.00u_PnP, F.Cu at (152.4, 57.1)
- added K_25: KEYSW, 122-LIB:SW_Hotswap_Kailh_MX_1.00u_PnP, F.Cu at (171.4, 57.1)
- added K_26: KEYSW, 122-LIB:SW_Hotswap_Kailh_MX_1.00u_PnP, F.Cu at (204.8, 57.1)
- added K_27: KEYSW, 122-LIB:SW_Hotswap_Kailh_MX_1.00u_PnP, F.Cu at (223.8, 57.1)
- added K_28: KEYSW, 122-LIB:SW_Hotswap_Kailh_MX_1.00u_PnP, F.Cu at (242.9, 57.1)
- added K_29: KEYSW, 122-LIB:SW_Hotswap_Kailh_MX_1.00u_PnP, F.Cu at (261.9, 57.1)
- added K_3: KEYSW, 122-LIB:SW_Hotswap_Kailh_MX_1.00u_PnP, F.Cu at (95.2, 38.1)
- added K_30: KEYSW, 122-LIB:SW_Hotswap_Kailh_MX_1.00u_PnP, F.Cu at (281.0, 57.1)
- added K_31: KEYSW, 122-LIB:SW_Hotswap_Kailh_MX_1.00u_PnP, F.Cu at (300.0, 57.1)
- added K_32: KEYSW, 122-LIB:SW_Hotswap_Kailh_MX_1.00u_PnP, F.Cu at (333.4, 57.1)
- added K_33: KEYSW, 122-LIB:SW_Hotswap_Kailh_MX_1.00u_PnP, F.Cu at (352.4, 57.1)
- added K_34: KEYSW, 122-LIB:SW_Hotswap_Kailh_MX_1.00u_PnP, F.Cu at (371.5, 57.1)
- added K_35: KEYSW, 122-LIB:SW_Hotswap_Kailh_MX_1.00u_PnP, F.Cu at (390.5, 57.1)
- added K_36: KEYSW, 122-LIB:SW_Hotswap_Kailh_MX_1.00u_PnP, F.Cu at (409.6, 57.1)
- added K_37: KEYSW, 122-LIB:SW_Hotswap_Kailh_MX_1.00u_PnP, F.Cu at (428.6, 57.1)
- added K_38: KEYSW, 122-LIB:SW_Hotswap_Kailh_MX_1.00u_PnP, F.Cu at (38.1, 85.7)
- added K_39: KEYSW, 122-LIB:SW_Hotswap_Kailh_MX_1.00u_PnP, F.Cu at (57.1, 85.7)
- added K_4: KEYSW, 122-LIB:SW_Hotswap_Kailh_MX_1.00u_PnP, F.Cu at (114.3, 38.1)
- added K_40: KEYSW, 122-LIB:SW_Hotswap_Kailh_MX_1.00u_PnP, F.Cu at (76.2, 85.7)
- added K_41: KEYSW, 122-LIB:SW_Hotswap_Kailh_MX_1.00u_PnP, F.Cu at (95.2, 85.7)
- added K_42: KEYSW, 122-LIB:SW_Hotswap_Kailh_MX_1.00u_PnP, F.Cu at (119.1, 85.7)
- added K_43: KEYSW, 122-LIB:SW_Hotswap_Kailh_MX_1.00u_PnP, F.Cu at (138.1, 85.7)
- added K_44: KEYSW, 122-LIB:SW_Hotswap_Kailh_MX_1.00u_PnP, F.Cu at (157.2, 85.7)
- added K_45: KEYSW, 122-LIB:SW_Hotswap_Kailh_MX_1.00u_PnP, F.Cu at (176.2, 85.7)
- added K_46: KEYSW, 122-LIB:SW_Hotswap_Kailh_MX_1.00u_PnP, F.Cu at (195.3, 85.7)
- added K_47: KEYSW, 122-LIB:SW_Hotswap_Kailh_MX_1.00u_PnP, F.Cu at (214.3, 85.7)
- added K_48: KEYSW, 122-LIB:SW_Hotswap_Kailh_MX_1.00u_PnP, F.Cu at (233.4, 85.7)
- added K_49: KEYSW, 122-LIB:SW_Hotswap_Kailh_MX_1.00u_PnP, F.Cu at (252.4, 85.7)
- added K_5: KEYSW, 122-LIB:SW_Hotswap_Kailh_MX_1.00u_PnP, F.Cu at (133.3, 38.1)
- added K_50: KEYSW, 122-LIB:SW_Hotswap_Kailh_MX_1.00u_PnP, F.Cu at (271.5, 85.7)
- added K_51: KEYSW, 122-LIB:SW_Hotswap_Kailh_MX_1.00u_PnP, F.Cu at (290.5, 85.7)
- added K_52: KEYSW, 122-LIB:SW_Hotswap_Kailh_MX_1.00u_PnP, F.Cu at (309.6, 85.7)
- added K_53: KEYSW, 122-LIB:SW_Hotswap_Kailh_MX_1.00u_PnP, F.Cu at (328.6, 85.7)
- added K_54: KEYSW, 122-LIB:SW_Hotswap_Kailh_MX_1.00u_PnP, F.Cu at (347.7, 85.7)
- added K_55: KEYSW, 122-LIB:SW_Hotswap_Kailh_MX_1.00u_PnP, F.Cu at (376.2, 85.7)
- added K_56: KEYSW, 122-LIB:SW_Hotswap_Kailh_MX_1.00u_PnP, F.Cu at (409.6, 85.7)
- added K_57: KEYSW, 122-LIB:SW_Hotswap_Kailh_MX_1.00u_PnP, F.Cu at (428.6, 85.7)
- added K_58: KEYSW, 122-LIB:SW_Hotswap_Kailh_MX_1.00u_PnP, F.Cu at (447.7, 85.7)
- added K_59: KEYSW, 122-LIB:SW_Hotswap_Kailh_MX_1.00u_PnP, F.Cu at (38.1, 104.8)
- added K_6: KEYSW, 122-LIB:SW_Hotswap_Kailh_MX_1.00u_PnP, F.Cu at (152.4, 38.1)
- added K_60: KEYSW, 122-LIB:SW_Hotswap_Kailh_MX_1.00u_PnP, F.Cu at (57.1, 104.8)
- added K_61: KEYSW, 122-LIB:SW_Hotswap_Kailh_MX_1.00u_PnP, F.Cu at (76.2, 104.8)
- added K_62: KEYSW, 122-LIB:SW_Hotswap_Kailh_MX_1.00u_PnP, F.Cu at (95.2, 104.8)
- added K_63: KEYSW, 122-LIB:SW_Hotswap_Kailh_MX_1.00u_PnP, F.Cu at (123.8, 104.8)
- added K_64: KEYSW, 122-LIB:SW_Hotswap_Kailh_MX_1.00u_PnP, F.Cu at (147.6, 104.8)
- added K_65: KEYSW, 122-LIB:SW_Hotswap_Kailh_MX_1.00u_PnP, F.Cu at (166.7, 104.8)
- added K_66: KEYSW, 122-LIB:SW_Hotswap_Kailh_MX_1.00u_PnP, F.Cu at (185.7, 104.8)
- added K_67: KEYSW, 122-LIB:SW_Hotswap_Kailh_MX_1.00u_PnP, F.Cu at (204.8, 104.8)
- added K_68: KEYSW, 122-LIB:SW_Hotswap_Kailh_MX_1.00u_PnP, F.Cu at (223.8, 104.8)
- added K_69: KEYSW, 122-LIB:SW_Hotswap_Kailh_MX_1.00u_PnP, F.Cu at (242.9, 104.8)
- added K_7: KEYSW, 122-LIB:SW_Hotswap_Kailh_MX_1.00u_PnP, F.Cu at (171.4, 38.1)
- added K_70: KEYSW, 122-LIB:SW_Hotswap_Kailh_MX_1.00u_PnP, F.Cu at (261.9, 104.8)
- added K_71: KEYSW, 122-LIB:SW_Hotswap_Kailh_MX_1.00u_PnP, F.Cu at (281.0, 104.8)
- added K_72: KEYSW, 122-LIB:SW_Hotswap_Kailh_MX_1.00u_PnP, F.Cu at (300.0, 104.8)
- added K_73: KEYSW, 122-LIB:SW_Hotswap_Kailh_MX_1.00u_PnP, F.Cu at (319.1, 104.8)
- added K_74: KEYSW, 122-LIB:SW_Hotswap_Kailh_MX_1.00u_PnP, F.Cu at (338.1, 104.8)
- added K_75: KEYSW, 122-LIB:SW_Hotswap_Kailh_MX_1.00u_PnP, F.Cu at (357.2, 104.8)
- added K_76: KEYSW, 122-LIB:SW_Hotswap_Kailh_MX_1.00u_PnP, F.Cu at (381.0, 104.8)
- added K_77: KEYSW, 122-LIB:SW_Hotswap_Kailh_MX_1.00u_PnP, F.Cu at (409.6, 104.8)
- added K_78: KEYSW, 122-LIB:SW_Hotswap_Kailh_MX_1.00u_PnP, F.Cu at (428.6, 104.8)
- added K_79: KEYSW, 122-LIB:SW_Hotswap_Kailh_MX_1.00u_PnP, F.Cu at (447.7, 104.8)
- added K_8: KEYSW, 122-LIB:SW_Hotswap_Kailh_MX_1.00u_PnP, F.Cu at (204.8, 38.1)
- added K_80: KEYSW, 122-LIB:SW_Hotswap_Kailh_MX_1.00u_PnP, F.Cu at (38.1, 123.8)
- added K_81: KEYSW, 122-LIB:SW_Hotswap_Kailh_MX_1.00u_PnP, F.Cu at (57.1, 123.8)
- added K_82: KEYSW, 122-LIB:SW_Hotswap_Kailh_MX_1.00u_PnP, F.Cu at (76.2, 123.8)
- added K_83: KEYSW, 122-LIB:SW_Hotswap_Kailh_MX_1.00u_PnP, F.Cu at (95.2, 123.8)
- added K_84: KEYSW, 122-LIB:SW_Hotswap_Kailh_MX_1.00u_PnP, F.Cu at (126.2, 123.8)
- added K_85: KEYSW, 122-LIB:SW_Hotswap_Kailh_MX_1.00u_PnP, F.Cu at (152.4, 123.8)
- added K_86: KEYSW, 122-LIB:SW_Hotswap_Kailh_MX_1.00u_PnP, F.Cu at (171.4, 123.8)
- added K_87: KEYSW, 122-LIB:SW_Hotswap_Kailh_MX_1.00u_PnP, F.Cu at (190.5, 123.8)
- added K_88: KEYSW, 122-LIB:SW_Hotswap_Kailh_MX_1.00u_PnP, F.Cu at (209.6, 123.8)
- added K_89: KEYSW, 122-LIB:SW_Hotswap_Kailh_MX_1.00u_PnP, F.Cu at (228.6, 123.8)
- added K_9: KEYSW, 122-LIB:SW_Hotswap_Kailh_MX_1.00u_PnP, F.Cu at (223.8, 38.1)
- added K_90: KEYSW, 122-LIB:SW_Hotswap_Kailh_MX_1.00u_PnP, F.Cu at (247.7, 123.8)
- added K_91: KEYSW, 122-LIB:SW_Hotswap_Kailh_MX_1.00u_PnP, F.Cu at (266.7, 123.8)
- added K_92: KEYSW, 122-LIB:SW_Hotswap_Kailh_MX_1.00u_PnP, F.Cu at (285.8, 123.8)
- added K_93: KEYSW, 122-LIB:SW_Hotswap_Kailh_MX_1.00u_PnP, F.Cu at (304.8, 123.8)
- added K_94: KEYSW, 122-LIB:SW_Hotswap_Kailh_MX_1.00u_PnP, F.Cu at (323.9, 123.8)
- added K_95: KEYSW, 122-LIB:SW_Hotswap_Kailh_MX_1.00u_PnP, F.Cu at (342.9, 123.8)
- added K_96: KEYSW, 122-LIB:SW_Hotswap_Kailh_MX_1.00u_PnP, F.Cu at (373.9, 123.8)
- added K_97: KEYSW, 122-LIB:SW_Hotswap_Kailh_MX_1.00u_PnP, F.Cu at (409.6, 123.8)
- added K_98: KEYSW, 122-LIB:SW_Hotswap_Kailh_MX_1.00u_PnP, F.Cu at (428.6, 123.8)
- added K_99: KEYSW, 122-LIB:SW_Hotswap_Kailh_MX_1.00u_PnP, F.Cu at (447.7, 123.8)
- added R1: 1k, Resistor_SMD:R_0402_1005Metric_Pad0.72x0.64mm_HandSolder, F.Cu at (-54.7, 127.0)
- added R10: 27, Resistor_SMD:R_0402_1005Metric_Pad0.72x0.64mm_HandSolder, F.Cu at (-51.4, 133.0)
- added R2: 10kR, Resistor_SMD:R_0402_1005Metric_Pad0.72x0.64mm_HandSolder, F.Cu at (-54.7, 129.0)
- added R3: 1k, Resistor_SMD:R_0402_1005Metric_Pad0.72x0.64mm_HandSolder, F.Cu at (-54.7, 131.0)
- added R4: 5.1kR, Resistor_SMD:R_0402_1005Metric_Pad0.72x0.64mm_HandSolder, F.Cu at (-54.7, 133.0)
- added R5: 5.1kR, Resistor_SMD:R_0402_1005Metric_Pad0.72x0.64mm_HandSolder, F.Cu at (-54.7, 135.0)
- added R6: 4.7kR, Resistor_SMD:R_0402_1005Metric_Pad0.72x0.64mm_HandSolder, F.Cu at (-54.7, 136.9)
- added R7: 100R, Resistor_SMD:R_0402_1005Metric_Pad0.72x0.64mm_HandSolder, F.Cu at (-51.4, 127.0)
- added R8: 100R, Resistor_SMD:R_0402_1005Metric_Pad0.72x0.64mm_HandSolder, F.Cu at (-51.4, 129.0)
- added R9: 27, Resistor_SMD:R_0402_1005Metric_Pad0.72x0.64mm_HandSolder, F.Cu at (-51.4, 131.0)
- added SW1: BOOTSEL, Button_Switch_SMD:SW_SPST_PTS810, F.Cu at (-37.7, 135.3)
- added SW2: RESET, Button_Switch_SMD:SW_SPST_PTS810, F.Cu at (-37.7, 140.1)
- added U1: W25Q128JVS, Package_SO:SOIC-8_5.3x5.3mm_P1.27mm, F.Cu at (-35.9, 129.5)
- added U2: NCP1117-3.3_SOT223, Package_TO_SOT_SMD:SOT-223-3_TabPin2, F.Cu at (-39.7, 120.2)
- added U3: RP2040, 122-LIB:RP2040, F.Cu at (-45.4, 130.4)
- added Y1: ABM8-272-T3, Crystal:Crystal_SMD_3225-4Pin_3.2x2.5mm, F.Cu at (-53.7, 140.2)
Other:
- board outline added: 428.7 x 147.7 mm

Commit message: Added updated files
Parts:
- J2: value Conn_01x03 -> DEBUG PROBE PORT
- R10, R9: value 27 -> 27R
- moved U3 24.4 mm to (-44.4, 154.7), turned to -45 degrees
Connections:
- U3 pad 1: unconnected-(U3-IOVDD-Pad1) -> +3V3
- U3 pad 10: unconnected-(U3-IOVDD-Pad10) -> +3V3
- U3 pad 22: unconnected-(U3-IOVDD-Pad22) -> +3V3
- U3 pad 23: unconnected-(U3-DVDD-Pad23) -> +1V1
- U3 pad 33: unconnected-(U3-IOVDD-Pad33) -> +3V3
- U3 pad 42: unconnected-(U3-IOVDD-Pad42) -> +3V3
- U3 pad 43: unconnected-(U3-ADC_AVDD-Pad43) -> +3V3
- U3 pad 44: unconnected-(U3-VREG_IN-Pad44) -> +3V3
- U3 pad 45: unconnected-(U3-VREG_VOUT-Pad45) -> +1V1
- U3 pad 48: unconnected-(U3-USB_VDD-Pad48) -> +3V3
- U3 pad 49: unconnected-(U3-IOVDD-Pad49) -> +3V3
- U3 pad 50: unconnected-(U3-DVDD-Pad50) -> +1V1
