File: V2/1800122-V2.kicad_pcb (KiCad board)
At the start: 2 copper layers, 428.7 x 147.7 mm, 279 parts, among them J1 USB_C_Receptacle_USB2.0_16P, J2 DEBUG PROBE PORT, SW1 BOOTSEL, SW2 RESET, U1 W25Q128JVS, U2 NCP1117-3.3_SOT223, U3 RP2040, Y1 ABM8-272-T3

Commit message: Fixes + new files
Added RP2040 docs, fixed diodes in key matrix schematic, assigned RP2040 footprint to KiCAD stock QFN-56 7x7 package and made the BOOTSEL and RESET buttons smaller format.
Parts:
- added C10: 100n, Capacitor_SMD:C_01005_0402Metric, F.Cu at (-16.6, 11.8)
- added C11: 100n, Capacitor_SMD:C_01005_0402Metric, F.Cu at (-16.6, 13.5)
- added C12: 100n, Capacitor_SMD:C_01005_0402Metric, F.Cu at (-16.6, 15.1)
- added C13: 100n, Capacitor_SMD:C_01005_0402Metric, F.Cu at (-16.6, 16.8)
- added C14: 100n, Capacitor_SMD:C_01005_0402Metric, F.Cu at (-16.6, 18.4)
- added C15: 100n, Capacitor_SMD:C_01005_0402Metric, F.Cu at (-14.4, 8.53)
- added C16: 100n, Capacitor_SMD:C_01005_0402Metric, F.Cu at (-14.4, 10.2)
- added C6: 1u, Capacitor_SMD:C_01005_0402Metric, F.Cu at (-18.9, 16.8)
- added C7: 1u, Capacitor_SMD:C_01005_0402Metric, F.Cu at (-18.9, 18.4)
- added C8: 100n, Capacitor_SMD:C_01005_0402Metric, F.Cu at (-16.6, 8.53)
- added C9: 100n, Capacitor_SMD:C_01005_0402Metric, F.Cu at (-16.6, 10.2)
- C1, C2, C3, C4, C5: footprint Capacitor_SMD:C_0402_1005Metric_Pad0.74x0.62mm_HandSolder -> Capacitor_SMD:C_01005_0402Metric
- D_92, D_93, D_98, D_99: moved to B.Cu
- R1, R10, R2, R3, R4, R5, R6, R7, R8, R9: footprint Resistor_SMD:R_0402_1005Metric_Pad0.72x0.64mm_HandSolder -> Resistor_SMD:R_01005_0402Metric
- SW1, SW2: footprint Button_Switch_SMD:SW_SPST_PTS810 -> Button_Switch_SMD:SW_SPST_B3U-1000P
- moved D_99 461.2 mm to (454.0, 132.8), turned to 90 degrees
- moved D_98 442.3 mm to (435.0, 132.8), turned to 90 degrees
- moved D_93 324.3 mm to (311.1, 132.8), turned to 90 degrees
- moved D_92 305.2 mm to (292.1, 132.8), turned to 90 degrees
- moved U3 135.7 mm to (-25.5, 20.4), turned to 0 degrees
- moved R6 135.3 mm to (-12.1, 8.53)
- moved J2 132.7 mm to (-7.07, 11.5)
- moved U1 130.3 mm to (-13.0, 1.25)
- moved R10 124.2 mm to (-12.1, 15.1)
- moved Y1 124.1 mm to (-17.4, 21.5)
- moved R9 123.9 mm to (-12.1, 13.5)
- moved R8 123.6 mm to (-12.1, 11.8)
- moved R5 123.3 mm to (-14.4, 18.4)
- moved R7 123.2 mm to (-12.1, 10.2)
- moved R4 123.0 mm to (-14.4, 16.8)
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Connections:
- D_92 pad 2: unconnected-(D_92-A-Pad2) -> Net-(D_92-A)
- D_93 pad 2: unconnected-(D_93-A-Pad2) -> Net-(D_93-A)
- D_98 pad 2: unconnected-(D_98-A-Pad2) -> Net-(D_98-A)
- D_99 pad 2: unconnected-(D_99-A-Pad2) -> Net-(D_99-A)
- J2 pad MP: (no net) -> unconnected-(J2-PadMP)
- K_92 pad 1: unconnected-(K_92-COL-Pad1) -> col14
- K_92 pad 2: unconnected-(K_92-ROW-Pad2) -> Net-(D_92-A)
- K_93 pad 1: unconnected-(K_93-COL-Pad1) -> col14
- K_93 pad 2: unconnected-(K_93-ROW-Pad2) -> Net-(D_93-A)
- K_98 pad 1: unconnected-(K_98-COL-Pad1) -> col15
- K_98 pad 2: unconnected-(K_98-ROW-Pad2) -> Net-(D_98-A)
- K_99 pad 1: unconnected-(K_99-COL-Pad1) -> col15
- K_99 pad 2: unconnected-(K_99-ROW-Pad2) -> Net-(D_99-A)
Other:
- board outline removed

Commit message: Updated KiCAD layout
Parts:
- C10, C8: value 100n -> 1u
- C6, C7: value 1u -> 100n
- J2: moved to B.Cu
- R6: value 4.7kR -> 100R
- R8: value 100R -> 4.7kR
- moved U2 145.9 mm to (115.4, 51.9), turned to -90 degrees
- moved J1 135.4 mm to (104.6, 45.2), turned to 180 degrees
- moved J2 128.2 mm to (83.0, 102.7), turned to 90 degrees
- moved SW1 111.0 mm to (71.6, 95.4)
- moved SW2 110.7 mm to (71.6, 99.7)
- moved U1 105.7 mm to (39.4, 93.1), turned to -45 degrees
- moved U3 100.1 mm to (33.8, 101.0), turned to -45 degrees
- moved R3 99.6 mm to (30.3, 104.2), turned to -135 degrees
- moved Y1 95.2 mm to (27.4, 105.5), turned to -45 degrees
- moved C1 78.3 mm to (29.9, 69.8)
- moved C10 78.3 mm to (32.1, 73.1)
- moved C11 78.3 mm to (32.1, 74.8)
- moved C12 78.3 mm to (32.1, 76.4)
- moved C13 78.3 mm to (32.1, 78.1)
- moved C14 78.3 mm to (32.1, 79.7)
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Connections:
- C7 pad 1: +3V3 -> +1V1
- C9 pad 1: +1V1 -> +3V3
- R6 pad 1: +3V3 -> /SWCLK
- R6 pad 2: Net-(U3-RUN) -> Net-(U3-SWCLK)
- R7 pad 1: /SWCLK -> /SWD
- R7 pad 2: Net-(U3-SWCLK) -> Net-(U3-SWD)
- R8 pad 1: /SWD -> +3V3
- R8 pad 2: Net-(U3-SWD) -> Net-(U3-RUN)
Routing:
- net Net-(D_74-A): track 0.00 -> 31.0 mm
- net Net-(D_97-A): track 0.00 -> 31.0 mm
- net Net-(D_91-A): track 0.00 -> 31.0 mm
- net Net-(D_77-A): track 0.00 -> 31.0 mm
- net Net-(D_69-A): track 0.00 -> 31.0 mm
- net Net-(D_92-A): track 0.00 -> 31.0 mm
- net Net-(D_78-A): track 0.00 -> 31.0 mm
- net Net-(D_70-A): track 0.00 -> 31.0 mm
- net Net-(D_98-A): track 0.00 -> 31.0 mm
- net Net-(D_87-A): track 0.00 -> 31.0 mm
- net Net-(D_65-A): track 0.00 -> 31.0 mm
- net Net-(D_81-A): track 0.00 -> 31.0 mm
- net Net-(D_80-A): track 0.00 -> 31.0 mm
- net Net-(D_59-A): track 0.00 -> 31.0 mm
- net Net-(D_60-A): track 0.00 -> 31.0 mm
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Other:
- board text added: "KEYSWITCH ORIGIN FROM UPPER LEFT EDGE OF OUTLINE X +8.575 Y -4.575"

Commit message: Added PnP for plated thru holes + literature
Parts:
- K_1, K_128, K_94: footprint 122-LIB:SW_Hotswap_Kailh_MX_1.00u_PnP -> 122-LIB:SW_Hotswap_Kailh_MX_Plated_1.00u_PnP
- K_10: renamed from K_64; footprint 122-LIB:SW_Hotswap_Kailh_MX_1.00u_PnP -> 122-LIB:SW_Hotswap_Kailh_MX_Plated_1.00u_PnP
- K_100: renamed from K_5; footprint 122-LIB:SW_Hotswap_Kailh_MX_1.00u_PnP -> 122-LIB:SW_Hotswap_Kailh_MX_Plated_1.00u_PnP
- K_101: renamed from K_10; footprint 122-LIB:SW_Hotswap_Kailh_MX_1.00u_PnP -> 122-LIB:SW_Hotswap_Kailh_MX_Plated_1.00u_PnP
- K_102: renamed from K_16; footprint 122-LIB:SW_Hotswap_Kailh_MX_1.00u_PnP -> 122-LIB:SW_Hotswap_Kailh_MX_Plated_1.00u_PnP
- K_103: renamed from K_23; footprint 122-LIB:SW_Hotswap_Kailh_MX_1.00u_PnP -> 122-LIB:SW_Hotswap_Kailh_MX_Plated_1.00u_PnP
- K_104: renamed from K_29; footprint 122-LIB:SW_Hotswap_Kailh_MX_1.00u_PnP -> 122-LIB:SW_Hotswap_Kailh_MX_Plated_1.00u_PnP
- K_105: renamed from K_36; footprint 122-LIB:SW_Hotswap_Kailh_MX_1.00u_PnP -> 122-LIB:SW_Hotswap_Kailh_MX_Plated_1.00u_PnP
- K_106: renamed from K_43; footprint 122-LIB:SW_Hotswap_Kailh_MX_1.00u_PnP -> 122-LIB:SW_Hotswap_Kailh_MX_Plated_1.00u_PnP
- K_107: renamed from K_50; footprint 122-LIB:SW_Hotswap_Kailh_MX_1.00u_PnP -> 122-LIB:SW_Hotswap_Kailh_MX_Plated_1.00u_PnP
- K_108: renamed from K_57; footprint 122-LIB:SW_Hotswap_Kailh_MX_1.00u_PnP -> 122-LIB:SW_Hotswap_Kailh_MX_Plated_1.00u_PnP
- K_109: renamed from K_63; footprint 122-LIB:SW_Hotswap_Kailh_MX_1.00u_PnP -> 122-LIB:SW_Hotswap_Kailh_MX_Plated_1.00u_PnP
- K_11: renamed from K_71; footprint 122-LIB:SW_Hotswap_Kailh_MX_1.00u_PnP -> 122-LIB:SW_Hotswap_Kailh_MX_Plated_1.00u_PnP
- K_110: renamed from K_69; footprint 122-LIB:SW_Hotswap_Kailh_MX_1.00u_PnP -> 122-LIB:SW_Hotswap_Kailh_MX_Plated_1.00u_PnP
- K_111: renamed from K_76; footprint 122-LIB:SW_Hotswap_Kailh_MX_1.00u_PnP -> 122-LIB:SW_Hotswap_Kailh_MX_Plated_1.00u_PnP
- K_112: renamed from K_82; footprint 122-LIB:SW_Hotswap_Kailh_MX_1.00u_PnP -> 122-LIB:SW_Hotswap_Kailh_MX_Plated_1.00u_PnP
- K_113: renamed from K_88; footprint 122-LIB:SW_Hotswap_Kailh_MX_1.00u_PnP -> 122-LIB:SW_Hotswap_Kailh_MX_Plated_1.00u_PnP
- K_114: renamed from K_95; footprint 122-LIB:SW_Hotswap_Kailh_MX_1.00u_PnP -> 122-LIB:SW_Hotswap_Kailh_MX_Plated_1.00u_PnP
- K_115: renamed from K_101; footprint 122-LIB:SW_Hotswap_Kailh_MX_1.00u_PnP -> 122-LIB:SW_Hotswap_Kailh_MX_Plated_1.00u_PnP
- K_116: renamed from K_117; footprint 122-LIB:SW_Hotswap_Kailh_MX_1.00u_PnP -> 122-LIB:SW_Hotswap_Kailh_MX_Plated_1.00u_PnP
- K_117: renamed from K_6; footprint 122-LIB:SW_Hotswap_Kailh_MX_1.00u_PnP -> 122-LIB:SW_Hotswap_Kailh_MX_Plated_1.00u_PnP
- K_118: renamed from K_17; footprint 122-LIB:SW_Hotswap_Kailh_MX_1.00u_PnP -> 122-LIB:SW_Hotswap_Kailh_MX_Plated_1.00u_PnP
- K_119: renamed from K_30; footprint 122-LIB:SW_Hotswap_Kailh_MX_1.00u_PnP -> 122-LIB:SW_Hotswap_Kailh_MX_Plated_1.00u_PnP
- K_12: renamed from K_77; footprint 122-LIB:SW_Hotswap_Kailh_MX_1.00u_PnP -> 122-LIB:SW_Hotswap_Kailh_MX_Plated_1.00u_PnP
- K_120: renamed from K_37; footprint 122-LIB:SW_Hotswap_Kailh_MX_1.00u_PnP -> 122-LIB:SW_Hotswap_Kailh_MX_Plated_1.00u_PnP
- K_121: renamed from K_44; footprint 122-LIB:SW_Hotswap_Kailh_MX_1.00u_PnP -> 122-LIB:SW_Hotswap_Kailh_MX_Plated_1.00u_PnP
- K_122: renamed from K_51; footprint 122-LIB:SW_Hotswap_Kailh_MX_1.00u_PnP -> 122-LIB:SW_Hotswap_Kailh_MX_Plated_1.00u_PnP
- K_123: renamed from K_70; footprint 122-LIB:SW_Hotswap_Kailh_MX_1.00u_PnP -> 122-LIB:SW_Hotswap_Kailh_MX_Plated_1.00u_PnP
- K_124: renamed from K_89; footprint 122-LIB:SW_Hotswap_Kailh_MX_1.00u_PnP -> 122-LIB:SW_Hotswap_Kailh_MX_Plated_1.00u_PnP
- K_125: renamed from K_102; footprint 122-LIB:SW_Hotswap_Kailh_MX_1.00u_PnP -> 122-LIB:SW_Hotswap_Kailh_MX_Plated_1.00u_PnP
- K_126: renamed from K_118; footprint 122-LIB:SW_Hotswap_Kailh_MX_1.00u_PnP -> 122-LIB:SW_Hotswap_Kailh_MX_Plated_1.00u_PnP
- K_127: renamed from K_124; footprint 122-LIB:SW_Hotswap_Kailh_MX_1.00u_PnP -> 122-LIB:SW_Hotswap_Kailh_MX_Plated_1.00u_PnP
- K_13: renamed from K_83; footprint 122-LIB:SW_Hotswap_Kailh_MX_1.00u_PnP -> 122-LIB:SW_Hotswap_Kailh_MX_Plated_1.00u_PnP
- K_14: renamed from K_90; footprint 122-LIB:SW_Hotswap_Kailh_MX_1.00u_PnP -> 122-LIB:SW_Hotswap_Kailh_MX_Plated_1.00u_PnP
- K_15: renamed from K_96; footprint 122-LIB:SW_Hotswap_Kailh_MX_1.00u_PnP -> 122-LIB:SW_Hotswap_Kailh_MX_Plated_1.00u_PnP
- K_16: renamed from K_103; footprint 122-LIB:SW_Hotswap_Kailh_MX_1.00u_PnP -> 122-LIB:SW_Hotswap_Kailh_MX_Plated_1.00u_PnP
- K_17: renamed from K_108; footprint 122-LIB:SW_Hotswap_Kailh_MX_1.00u_PnP -> 122-LIB:SW_Hotswap_Kailh_MX_Plated_1.00u_PnP
- K_18: renamed from K_112; footprint 122-LIB:SW_Hotswap_Kailh_MX_1.00u_PnP -> 122-LIB:SW_Hotswap_Kailh_MX_Plated_1.00u_PnP
- K_19: renamed from K_119; footprint 122-LIB:SW_Hotswap_Kailh_MX_1.00u_PnP -> 122-LIB:SW_Hotswap_Kailh_MX_Plated_1.00u_PnP
- K_2: renamed from K_11; footprint 122-LIB:SW_Hotswap_Kailh_MX_1.00u_PnP -> 122-LIB:SW_Hotswap_Kailh_MX_Plated_1.00u_PnP
- K_20: renamed from K_12; footprint 122-LIB:SW_Hotswap_Kailh_MX_1.00u_PnP -> 122-LIB:SW_Hotswap_Kailh_MX_Plated_1.00u_PnP
- K_21: renamed from K_19; footprint 122-LIB:SW_Hotswap_Kailh_MX_1.00u_PnP -> 122-LIB:SW_Hotswap_Kailh_MX_Plated_1.00u_PnP
- K_22: renamed from K_25; footprint 122-LIB:SW_Hotswap_Kailh_MX_1.00u_PnP -> 122-LIB:SW_Hotswap_Kailh_MX_Plated_1.00u_PnP
- K_23: renamed from K_32; footprint 122-LIB:SW_Hotswap_Kailh_MX_1.00u_PnP -> 122-LIB:SW_Hotswap_Kailh_MX_Plated_1.00u_PnP
- K_24: renamed from K_39; footprint 122-LIB:SW_Hotswap_Kailh_MX_1.00u_PnP -> 122-LIB:SW_Hotswap_Kailh_MX_Plated_1.00u_PnP
- K_25: renamed from K_46; footprint 122-LIB:SW_Hotswap_Kailh_MX_1.00u_PnP -> 122-LIB:SW_Hotswap_Kailh_MX_Plated_1.00u_PnP
- K_26: renamed from K_53; footprint 122-LIB:SW_Hotswap_Kailh_MX_1.00u_PnP -> 122-LIB:SW_Hotswap_Kailh_MX_Plated_1.00u_PnP
- K_27: renamed from K_59; footprint 122-LIB:SW_Hotswap_Kailh_MX_1.00u_PnP -> 122-LIB:SW_Hotswap_Kailh_MX_Plated_1.00u_PnP
- K_28: renamed from K_65; footprint 122-LIB:SW_Hotswap_Kailh_MX_1.00u_PnP -> 122-LIB:SW_Hotswap_Kailh_MX_Plated_1.00u_PnP
- K_29: renamed from K_72; footprint 122-LIB:SW_Hotswap_Kailh_MX_1.00u_PnP -> 122-LIB:SW_Hotswap_Kailh_MX_Plated_1.00u_PnP
- K_3: renamed from K_18; footprint 122-LIB:SW_Hotswap_Kailh_MX_1.00u_PnP -> 122-LIB:SW_Hotswap_Kailh_MX_Plated_1.00u_PnP
- K_30: renamed from K_78; footprint 122-LIB:SW_Hotswap_Kailh_MX_1.00u_PnP -> 122-LIB:SW_Hotswap_Kailh_MX_Plated_1.00u_PnP
- K_31: renamed from K_84; footprint 122-LIB:SW_Hotswap_Kailh_MX_1.00u_PnP -> 122-LIB:SW_Hotswap_Kailh_MX_Plated_1.00u_PnP
- K_32: renamed from K_91; footprint 122-LIB:SW_Hotswap_Kailh_MX_1.00u_PnP -> 122-LIB:SW_Hotswap_Kailh_MX_Plated_1.00u_PnP
- K_33: renamed from K_97; footprint 122-LIB:SW_Hotswap_Kailh_MX_1.00u_PnP -> 122-LIB:SW_Hotswap_Kailh_MX_Plated_1.00u_PnP
- K_34: renamed from K_104; footprint 122-LIB:SW_Hotswap_Kailh_MX_1.00u_PnP -> 122-LIB:SW_Hotswap_Kailh_MX_Plated_1.00u_PnP
- K_35: renamed from K_109; footprint 122-LIB:SW_Hotswap_Kailh_MX_1.00u_PnP -> 122-LIB:SW_Hotswap_Kailh_MX_Plated_1.00u_PnP
- K_36: renamed from K_113; footprint 122-LIB:SW_Hotswap_Kailh_MX_1.00u_PnP -> 122-LIB:SW_Hotswap_Kailh_MX_Plated_1.00u_PnP
- K_37: renamed from K_120; footprint 122-LIB:SW_Hotswap_Kailh_MX_1.00u_PnP -> 122-LIB:SW_Hotswap_Kailh_MX_Plated_1.00u_PnP
- K_38: renamed from K_2; footprint 122-LIB:SW_Hotswap_Kailh_MX_1.00u_PnP -> 122-LIB:SW_Hotswap_Kailh_MX_Plated_1.00u_PnP
- K_39: renamed from K_7; footprint 122-LIB:SW_Hotswap_Kailh_MX_1.00u_PnP -> 122-LIB:SW_Hotswap_Kailh_MX_Plated_1.00u_PnP
- K_4: renamed from K_24; footprint 122-LIB:SW_Hotswap_Kailh_MX_1.00u_PnP -> 122-LIB:SW_Hotswap_Kailh_MX_Plated_1.00u_PnP
- K_40: renamed from K_13; footprint 122-LIB:SW_Hotswap_Kailh_MX_1.00u_PnP -> 122-LIB:SW_Hotswap_Kailh_MX_Plated_1.00u_PnP
- K_41: renamed from K_20; footprint 122-LIB:SW_Hotswap_Kailh_MX_1.00u_PnP -> 122-LIB:SW_Hotswap_Kailh_MX_Plated_1.00u_PnP
- K_42: renamed from K_26; footprint 122-LIB:SW_Hotswap_Kailh_MX_1.00u_PnP -> 122-LIB:SW_Hotswap_Kailh_MX_Plated_1.00u_PnP
- K_43: renamed from K_33; footprint 122-LIB:SW_Hotswap_Kailh_MX_1.00u_PnP -> 122-LIB:SW_Hotswap_Kailh_MX_Plated_1.00u_PnP
- K_44: renamed from K_40; footprint 122-LIB:SW_Hotswap_Kailh_MX_1.00u_PnP -> 122-LIB:SW_Hotswap_Kailh_MX_Plated_1.00u_PnP
- K_45: renamed from K_47; footprint 122-LIB:SW_Hotswap_Kailh_MX_1.00u_PnP -> 122-LIB:SW_Hotswap_Kailh_MX_Plated_1.00u_PnP
- K_46: renamed from K_54; footprint 122-LIB:SW_Hotswap_Kailh_MX_1.00u_PnP -> 122-LIB:SW_Hotswap_Kailh_MX_Plated_1.00u_PnP
- K_47: renamed from K_60; footprint 122-LIB:SW_Hotswap_Kailh_MX_1.00u_PnP -> 122-LIB:SW_Hotswap_Kailh_MX_Plated_1.00u_PnP
- K_48: renamed from K_66; footprint 122-LIB:SW_Hotswap_Kailh_MX_1.00u_PnP -> 122-LIB:SW_Hotswap_Kailh_MX_Plated_1.00u_PnP
- K_49: renamed from K_73; footprint 122-LIB:SW_Hotswap_Kailh_MX_1.00u_PnP -> 122-LIB:SW_Hotswap_Kailh_MX_Plated_1.00u_PnP
- K_5: renamed from K_31; footprint 122-LIB:SW_Hotswap_Kailh_MX_1.00u_PnP -> 122-LIB:SW_Hotswap_Kailh_MX_Plated_1.00u_PnP
- K_50: renamed from K_79; footprint 122-LIB:SW_Hotswap_Kailh_MX_1.00u_PnP -> 122-LIB:SW_Hotswap_Kailh_MX_Plated_1.00u_PnP
- K_51: renamed from K_85; footprint 122-LIB:SW_Hotswap_Kailh_MX_1.00u_PnP -> 122-LIB:SW_Hotswap_Kailh_MX_Plated_1.00u_PnP
- K_52: renamed from K_92; footprint 122-LIB:SW_Hotswap_Kailh_MX_1.00u_PnP -> 122-LIB:SW_Hotswap_Kailh_MX_Plated_1.00u_PnP
- K_53: renamed from K_98; footprint 122-LIB:SW_Hotswap_Kailh_MX_1.00u_PnP -> 122-LIB:SW_Hotswap_Kailh_MX_Plated_1.00u_PnP
- K_54: renamed from K_105; footprint 122-LIB:SW_Hotswap_Kailh_MX_1.00u_PnP -> 122-LIB:SW_Hotswap_Kailh_MX_Plated_1.00u_PnP
- K_55: renamed from K_110; footprint 122-LIB:SW_Hotswap_Kailh_MX_1.00u_PnP -> 122-LIB:SW_Hotswap_Kailh_MX_Plated_1.00u_PnP
- K_56: renamed from K_114; footprint 122-LIB:SW_Hotswap_Kailh_MX_1.00u_PnP -> 122-LIB:SW_Hotswap_Kailh_MX_Plated_1.00u_PnP
- K_57: renamed from K_121; footprint 122-LIB:SW_Hotswap_Kailh_MX_1.00u_PnP -> 122-LIB:SW_Hotswap_Kailh_MX_Plated_1.00u_PnP
- K_58: renamed from K_125; footprint 122-LIB:SW_Hotswap_Kailh_MX_1.00u_PnP -> 122-LIB:SW_Hotswap_Kailh_MX_Plated_1.00u_PnP
- K_59: renamed from K_3; footprint 122-LIB:SW_Hotswap_Kailh_MX_1.00u_PnP -> 122-LIB:SW_Hotswap_Kailh_MX_Plated_1.00u_PnP
- K_6: renamed from K_38; footprint 122-LIB:SW_Hotswap_Kailh_MX_1.00u_PnP -> 122-LIB:SW_Hotswap_Kailh_MX_Plated_1.00u_PnP
- K_60: renamed from K_8; footprint 122-LIB:SW_Hotswap_Kailh_MX_1.00u_PnP -> 122-LIB:SW_Hotswap_Kailh_MX_Plated_1.00u_PnP
- K_61: renamed from K_14; footprint 122-LIB:SW_Hotswap_Kailh_MX_1.00u_PnP -> 122-LIB:SW_Hotswap_Kailh_MX_Plated_1.00u_PnP
- K_62: renamed from K_21; footprint 122-LIB:SW_Hotswap_Kailh_MX_1.00u_PnP -> 122-LIB:SW_Hotswap_Kailh_MX_Plated_1.00u_PnP
- K_63: renamed from K_27; footprint 122-LIB:SW_Hotswap_Kailh_MX_1.00u_PnP -> 122-LIB:SW_Hotswap_Kailh_MX_Plated_1.00u_PnP
- K_64: renamed from K_34; footprint 122-LIB:SW_Hotswap_Kailh_MX_1.00u_PnP -> 122-LIB:SW_Hotswap_Kailh_MX_Plated_1.00u_PnP
- K_65: renamed from K_41; footprint 122-LIB:SW_Hotswap_Kailh_MX_1.00u_PnP -> 122-LIB:SW_Hotswap_Kailh_MX_Plated_1.00u_PnP
- K_66: renamed from K_48; footprint 122-LIB:SW_Hotswap_Kailh_MX_1.00u_PnP -> 122-LIB:SW_Hotswap_Kailh_MX_Plated_1.00u_PnP
- K_67: renamed from K_55; footprint 122-LIB:SW_Hotswap_Kailh_MX_1.00u_PnP -> 122-LIB:SW_Hotswap_Kailh_MX_Plated_1.00u_PnP
- K_68: renamed from K_61; footprint 122-LIB:SW_Hotswap_Kailh_MX_1.00u_PnP -> 122-LIB:SW_Hotswap_Kailh_MX_Plated_1.00u_PnP
- K_69: renamed from K_67; footprint 122-LIB:SW_Hotswap_Kailh_MX_1.00u_PnP -> 122-LIB:SW_Hotswap_Kailh_MX_Plated_1.00u_PnP
- K_7: renamed from K_45; footprint 122-LIB:SW_Hotswap_Kailh_MX_1.00u_PnP -> 122-LIB:SW_Hotswap_Kailh_MX_Plated_1.00u_PnP
- K_70: renamed from K_74; footprint 122-LIB:SW_Hotswap_Kailh_MX_1.00u_PnP -> 122-LIB:SW_Hotswap_Kailh_MX_Plated_1.00u_PnP
- K_71: renamed from K_80; footprint 122-LIB:SW_Hotswap_Kailh_MX_1.00u_PnP -> 122-LIB:SW_Hotswap_Kailh_MX_Plated_1.00u_PnP
- K_72: renamed from K_86; footprint 122-LIB:SW_Hotswap_Kailh_MX_1.00u_PnP -> 122-LIB:SW_Hotswap_Kailh_MX_Plated_1.00u_PnP
- K_73: renamed from K_93; footprint 122-LIB:SW_Hotswap_Kailh_MX_1.00u_PnP -> 122-LIB:SW_Hotswap_Kailh_MX_Plated_1.00u_PnP
- K_74: renamed from K_99; footprint 122-LIB:SW_Hotswap_Kailh_MX_1.00u_PnP -> 122-LIB:SW_Hotswap_Kailh_MX_Plated_1.00u_PnP
- K_75: renamed from K_106; footprint 122-LIB:SW_Hotswap_Kailh_MX_1.00u_PnP -> 122-LIB:SW_Hotswap_Kailh_MX_Plated_1.00u_PnP
- K_76: renamed from K_111; footprint 122-LIB:SW_Hotswap_Kailh_MX_1.00u_PnP -> 122-LIB:SW_Hotswap_Kailh_MX_Plated_1.00u_PnP
- K_77: renamed from K_115; footprint 122-LIB:SW_Hotswap_Kailh_MX_1.00u_PnP -> 122-LIB:SW_Hotswap_Kailh_MX_Plated_1.00u_PnP
- K_78: renamed from K_122; footprint 122-LIB:SW_Hotswap_Kailh_MX_1.00u_PnP -> 122-LIB:SW_Hotswap_Kailh_MX_Plated_1.00u_PnP
- K_79: renamed from K_126; footprint 122-LIB:SW_Hotswap_Kailh_MX_1.00u_PnP -> 122-LIB:SW_Hotswap_Kailh_MX_Plated_1.00u_PnP
- K_8: renamed from K_52; footprint 122-LIB:SW_Hotswap_Kailh_MX_1.00u_PnP -> 122-LIB:SW_Hotswap_Kailh_MX_Plated_1.00u_PnP
- K_80: renamed from K_4; footprint 122-LIB:SW_Hotswap_Kailh_MX_1.00u_PnP -> 122-LIB:SW_Hotswap_Kailh_MX_Plated_1.00u_PnP
- K_81: renamed from K_9; footprint 122-LIB:SW_Hotswap_Kailh_MX_1.00u_PnP -> 122-LIB:SW_Hotswap_Kailh_MX_Plated_1.00u_PnP
- K_82: renamed from K_15; footprint 122-LIB:SW_Hotswap_Kailh_MX_1.00u_PnP -> 122-LIB:SW_Hotswap_Kailh_MX_Plated_1.00u_PnP
- K_83: renamed from K_22; footprint 122-LIB:SW_Hotswap_Kailh_MX_1.00u_PnP -> 122-LIB:SW_Hotswap_Kailh_MX_Plated_1.00u_PnP
- K_84: renamed from K_28; footprint 122-LIB:SW_Hotswap_Kailh_MX_1.00u_PnP -> 122-LIB:SW_Hotswap_Kailh_MX_Plated_1.00u_PnP
- K_85: renamed from K_35; footprint 122-LIB:SW_Hotswap_Kailh_MX_1.00u_PnP -> 122-LIB:SW_Hotswap_Kailh_MX_Plated_1.00u_PnP
- K_86: renamed from K_42; footprint 122-LIB:SW_Hotswap_Kailh_MX_1.00u_PnP -> 122-LIB:SW_Hotswap_Kailh_MX_Plated_1.00u_PnP
- K_87: renamed from K_49; footprint 122-LIB:SW_Hotswap_Kailh_MX_1.00u_PnP -> 122-LIB:SW_Hotswap_Kailh_MX_Plated_1.00u_PnP
- K_88: renamed from K_56; footprint 122-LIB:SW_Hotswap_Kailh_MX_1.00u_PnP -> 122-LIB:SW_Hotswap_Kailh_MX_Plated_1.00u_PnP
- K_89: renamed from K_62; footprint 122-LIB:SW_Hotswap_Kailh_MX_1.00u_PnP -> 122-LIB:SW_Hotswap_Kailh_MX_Plated_1.00u_PnP
- K_9: renamed from K_58; footprint 122-LIB:SW_Hotswap_Kailh_MX_1.00u_PnP -> 122-LIB:SW_Hotswap_Kailh_MX_Plated_1.00u_PnP
- K_90: renamed from K_68; footprint 122-LIB:SW_Hotswap_Kailh_MX_1.00u_PnP -> 122-LIB:SW_Hotswap_Kailh_MX_Plated_1.00u_PnP
- K_91: renamed from K_75; footprint 122-LIB:SW_Hotswap_Kailh_MX_1.00u_PnP -> 122-LIB:SW_Hotswap_Kailh_MX_Plated_1.00u_PnP
- K_92: renamed from K_81; footprint 122-LIB:SW_Hotswap_Kailh_MX_1.00u_PnP -> 122-LIB:SW_Hotswap_Kailh_MX_Plated_1.00u_PnP
- K_93: renamed from K_87; footprint 122-LIB:SW_Hotswap_Kailh_MX_1.00u_PnP -> 122-LIB:SW_Hotswap_Kailh_MX_Plated_1.00u_PnP
- K_95: renamed from K_100; footprint 122-LIB:SW_Hotswap_Kailh_MX_1.00u_PnP -> 122-LIB:SW_Hotswap_Kailh_MX_Plated_1.00u_PnP
- K_96: renamed from K_107; footprint 122-LIB:SW_Hotswap_Kailh_MX_1.00u_PnP -> 122-LIB:SW_Hotswap_Kailh_MX_Plated_1.00u_PnP
- K_97: renamed from K_116; footprint 122-LIB:SW_Hotswap_Kailh_MX_1.00u_PnP -> 122-LIB:SW_Hotswap_Kailh_MX_Plated_1.00u_PnP
- K_98: renamed from K_123; footprint 122-LIB:SW_Hotswap_Kailh_MX_1.00u_PnP -> 122-LIB:SW_Hotswap_Kailh_MX_Plated_1.00u_PnP
- K_99: renamed from K_127; footprint 122-LIB:SW_Hotswap_Kailh_MX_1.00u_PnP -> 122-LIB:SW_Hotswap_Kailh_MX_Plated_1.00u_PnP
- moved D_116 352.7 mm to (456.9, 183.1)
- moved K_116 352.7 mm to (450.5, 174.1)
- moved D_118 337.8 mm to (133.0, 197.4)
- moved K_118 337.8 mm to (126.7, 188.4)
- moved D_21 333.9 mm to (152.1, 92.6)
- moved K_21 333.9 mm to (145.7, 83.6)
- moved K_19 331.2 mm to (479.1, 64.6)
- moved D_19 331.2 mm to (485.4, 73.6)
- moved K_3 314.3 mm to (145.7, 64.6)
- moved D_3 314.3 mm to (152.1, 73.6)
- moved D_102 313.3 mm to (133.0, 178.3)
- moved K_102 313.3 mm to (126.7, 169.3)
- moved D_115 307.2 mm to (421.2, 178.3)
- moved K_115 307.2 mm to (414.8, 169.3)
- moved D_95 305.4 mm to (399.7, 159.3)
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- renumbered C3 to C1, C15 to C10, C16 to C11, C8 to C12, C10 to C13, C4 to C14, C1 to C15, C2 to C16, C5 to C2, C6 to C3, C7 to C4, C9 to C5, C11 to C6, C12 to C7, C13 to C8, C14 to C9, D_64 to D_10, D_5 to D_100, D_10 to D_101, D_16 to D_102, D_23 to D_103, D_29 to D_104, D_36 to D_105, D_43 to D_106, D_50 to D_107, D_57 to D_108, D_63 to D_109, D_71 to D_11, D_69 to D_110, D_76 to D_111, D_82 to D_112, D_88 to D_113, D_95 to D_114, D_101 to D_115, D_117 to D_116, D_6 to D_117, D_17 to D_118, D_30 to D_119, D_77 to D_12, D_37 to D_120, D_44 to D_121, D_51 to D_122, D_70 to D_123, D_89 to D_124, D_102 to D_125, D_118 to D_126, D_124 to D_127, D_83 to D_13, D_90 to D_14, D_96 to D_15, D_103 to D_16, D_108 to D_17, D_112 to D_18, D_119 to D_19, D_11 to D_2, D_12 to D_20, D_19 to D_21, D_25 to D_22, D_32 to D_23, D_39 to D_24, D_46 to D_25, D_53 to D_26, D_59 to D_27, D_65 to D_28, D_72 to D_29, D_18 to D_3, D_78 to D_30, D_84 to D_31, D_91 to D_32, D_97 to D_33, D_104 to D_34, D_109 to D_35, D_113 to D_36, D_120 to D_37, D_2 to D_38, D_7 to D_39, D_24 to D_4, D_13 to D_40, D_20 to D_41, D_26 to D_42, D_33 to D_43, D_40 to D_44, D_47 to D_45, D_54 to D_46, D_60 to D_47, D_66 to D_48, D_73 to D_49, D_31 to D_5, D_79 to D_50, D_85 to D_51, D_92 to D_52, D_98 to D_53, D_105 to D_54, D_110 to D_55, D_114 to D_56, D_121 to D_57, D_125 to D_58, D_3 to D_59, D_38 to D_6, D_8 to D_60, D_14 to D_61, D_21 to D_62, D_27 to D_63, D_34 to D_64, D_41 to D_65, D_48 to D_66, D_55 to D_67, D_61 to D_68, D_67 to D_69, D_45 to D_7, D_74 to D_70, D_80 to D_71, D_86 to D_72, D_93 to D_73, D_99 to D_74, D_106 to D_75, D_111 to D_76, D_115 to D_77, D_122 to D_78, D_126 to D_79, D_52 to D_8, D_4 to D_80, D_9 to D_81, D_15 to D_82, D_22 to D_83, D_28 to D_84, D_35 to D_85, D_42 to D_86, D_49 to D_87, D_56 to D_88, D_62 to D_89, D_58 to D_9, D_68 to D_90, D_75 to D_91, D_81 to D_92, D_87 to D_93, D_100 to D_95, D_107 to D_96, D_116 to D_97, D_123 to D_98, D_127 to D_99, R4 to R1, R8 to R10, R5 to R2, R2 to R3, R9 to R4, R10 to R5, R1 to R6, R3 to R7, R6 to R8, R7 to R9, U2 to U1, U1 to U2
Routing:
- net row4: track 0.00 -> 409.6 mm
- net row3: track 0.00 -> 409.6 mm
- net row2: track 0.00 -> 409.6 mm
- net row0: track 0.00 -> 390.5 mm
- net row5: track 0.00 -> 371.8 mm
- net row6: track 2.40 -> 373.4 mm
- net row1: track 0.00 -> 352.4 mm
- net Net-(D_77-A): track 28.6 -> 57.3 mm
- net Net-(D_98-A): track 28.6 -> 57.3 mm
- net Net-(D_74-A): track 28.6 -> 57.3 mm
- net Net-(D_97-A): track 28.6 -> 57.3 mm
- net Net-(D_78-A): track 28.6 -> 57.3 mm
- net Net-(D_56-A): track 28.6 -> 57.3 mm
- net Net-(D_57-A): track 28.6 -> 57.3 mm
- net Net-(D_19-A): track 28.6 -> 57.3 mm
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Other:
- board outline added: 450 x 167.8 mm
