File: V2/1800122-V2.kicad_pcb (KiCad board)
At the start: 2 copper layers, 450 x 167.8 mm, 290 parts, among them J1 USB_C_Receptacle_USB2.0_16P, J2 DEBUG PROBE PORT, SW1 BOOTSEL, SW2 RESET, U1 NCP1117-3.3_SOT223, U2 W25Q128JVS, U3 RP2040, Y1 ABM8-272-T3

Commit message: Added files
Made changes to schematic to use unified daughter board S1 layout
Parts:
- removed R1, R2: 5.1kR, Resistor_SMD:R_01005_0402Metric
- C1, C10, C11, C12, C13, C14, C15, C16, C2, C3, C4, C5, C6, C7, C8, C9: footprint Capacitor_SMD:C_01005_0402Metric -> Capacitor_SMD:C_0402_1005Metric
- J1: value USB_C_Receptacle_USB2.0_16P -> 78171-0004; footprint Connector_USB:USB_C_Receptacle_GCT_USB4105-xx-A_16P_TopMnt_Horizontal -> 122-LIB:PicoEZMate-Reinforced-Lite; moved to B.Cu
- R10, R3, R4, R5, R6, R7, R8, R9: footprint Resistor_SMD:R_01005_0402Metric -> Resistor_SMD:R_0402_1005Metric
- moved J1 109.1 mm to (53.2, 152.2)
- moved C9 20.0 mm to (36.4, 60.2)
- moved R3 16.0 mm to (27.8, 60.3)
- moved C14 15.7 mm to (39.3, 62.2)
- moved R4 15.3 mm to (27.8, 62.2)
- moved R5 15.1 mm to (27.8, 64.2)
- moved C13 14.8 mm to (39.3, 60.2)
- moved C2 14.3 mm to (30.7, 62.2)
- moved C3 13.9 mm to (30.7, 64.2)
- moved C4 13.6 mm to (30.7, 66.2)
- moved C1 12.9 mm to (30.7, 60.2)
- moved C6 12.7 mm to (33.5, 62.2)
- moved C7 12.3 mm to (33.5, 64.2)
- moved C8 12.0 mm to (33.5, 66.2)
- moved C5 11.3 mm to (33.5, 60.2)
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Routing:
- net Net-(D_76-A): track 57.3 -> 76.4 mm
- net Net-(D_70-A): track 57.3 -> 76.4 mm
- net Net-(D_98-A): track 57.3 -> 76.4 mm
- net Net-(D_69-A): track 57.3 -> 76.4 mm
- net Net-(D_97-A): track 57.3 -> 76.4 mm
- net Net-(D_74-A): track 57.3 -> 76.4 mm
- net Net-(D_96-A): track 57.3 -> 76.4 mm
- net Net-(D_92-A): track 57.3 -> 76.4 mm
- net Net-(D_91-A): track 57.3 -> 76.4 mm
- net Net-(D_78-A): track 57.3 -> 76.4 mm
- net Net-(D_75-A): track 57.3 -> 76.4 mm
- net Net-(D_84-A): track 57.3 -> 76.4 mm
- net Net-(D_83-A): track 57.3 -> 76.4 mm
- net Net-(D_82-A): track 57.3 -> 76.4 mm
- net Net-(D_77-A): track 57.3 -> 76.4 mm
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
Commit message: New library updates and changes to PnP footprints
Parts:
- moved D_1 3.49 mm to (97.4, 76.0)
- moved D_10 3.49 mm to (302.2, 76.0)
- moved D_100 3.49 mm to (97.4, 180.8)
- moved D_101 3.49 mm to (116.5, 180.8)
- moved D_103 3.49 mm to (154.6, 190.3)
- moved D_104 3.49 mm to (190.3, 180.8)
- moved D_105 3.49 mm to (221.2, 180.8)
- moved D_108 3.49 mm to (278.4, 180.8)
- moved D_109 3.49 mm to (297.4, 180.8)
- moved D_11 3.49 mm to (321.3, 76.0)
- moved D_110 3.49 mm to (316.5, 180.8)
- moved D_111 3.49 mm to (335.5, 180.8)
- moved D_113 3.49 mm to (373.6, 180.8)
- moved D_114 3.49 mm to (392.7, 180.8)
- moved D_115 3.49 mm to (423.6, 180.8)
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Routing:
- net row4: track 409.6 -> 0.00 mm
- net row3: track 409.6 -> 0.00 mm
- net row2: track 409.6 -> 0.00 mm
- net row0: track 390.5 -> 0.00 mm
- net row6: track 373.4 -> 0.00 mm
- net row5: track 371.8 -> 0.00 mm
- net row1: track 352.4 -> 0.00 mm
- net Net-(D_76-A): track 76.4 -> 11.8 mm
- net Net-(D_70-A): track 76.4 -> 11.8 mm
- net Net-(D_98-A): track 76.4 -> 11.8 mm
- net Net-(D_78-A): track 76.4 -> 11.8 mm
- net Net-(D_75-A): track 76.4 -> 11.8 mm
- net Net-(D_92-A): track 76.4 -> 11.8 mm
- net Net-(D_69-A): track 76.4 -> 11.8 mm
- net Net-(D_74-A): track 76.4 -> 11.8 mm
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Other:
- board text added: "KEYSWITCH ORIGIN FROM UPPER LEFT EDGE OF OUTLINE X +8.915 Y -5.715"
- board text removed: "KEYSWITCH ORIGIN FROM UPPER LEFT EDGE OF OUTLINE X +8.575 Y -4.575"
