File: V2/1800122-V2.kicad_sch (KiCad schematic)
At the start: 23 parts, among them J1 USB_C_Receptacle_USB2.0_16P, J2 DEBUG PROBE PORT, SW1 BOOTSEL, SW2 RESET, U1 W25Q128JVS, U2 NCP1117-3.3_SOT223, U3 RP2040, Y1 ABM8-272-T3

Commit message: Fixes + new files
Added RP2040 docs, fixed diodes in key matrix schematic, assigned RP2040 footprint to KiCAD stock QFN-56 7x7 package and made the BOOTSEL and RESET buttons smaller format.
Parts:
- added C10, C11, C12, C13, C14, C15, C16, C8, C9: 100n, Capacitor_SMD:C_01005_0402Metric, symbol Device:C
- added C6, C7: 1u, Capacitor_SMD:C_01005_0402Metric, symbol Device:C
- C1, C2, C3, C4, C5: footprint Capacitor_SMD:C_0402_1005Metric_Pad0.74x0.62mm_HandSolder -> Capacitor_SMD:C_01005_0402Metric
- R1, R10, R2, R3, R4, R5, R6, R7, R8, R9: footprint Resistor_SMD:R_0402_1005Metric_Pad0.72x0.64mm_HandSolder -> Resistor_SMD:R_01005_0402Metric
- SW1, SW2: footprint Button_Switch_SMD:SW_SPST_PTS810 -> Button_Switch_SMD:SW_SPST_B3U-1000P
Connections:
- net +1V1: now also C6.1, C8.1, C9.1
- net +3V3: now also C10.1, C11.1, C12.1, C13.1, C14.1, C15.1, C16.1, C7.1
- net GND: now also C10.2, C11.2, C12.2, C13.2, C14.2, C15.2, C16.2, C6.2, C7.2, C8.2, C9.2
Other:
- note added: "10% 16V X5R M1005"
- note added: "10% 25V X7R M1005"
- note added: "LCSC: C231329"
- note added: "Place C6 close to pin 45"
- note added: "Place C7 close to pin 44"
- moved on the sheet: R10, R6, R7, R8, R9, SW2, U3

Commit message: Updated KiCAD layout
Parts:
- renumbered C7 to C10, C8 to C6, C9 to C7, C6 to C8, C10 to C9, R7 to R6, R8 to R7, R6 to R8

Commit message: Added PnP for plated thru holes + literature
Parts:
- renumbered C3 to C1, C15 to C10, C16 to C11, C8 to C12, C10 to C13, C4 to C14, C1 to C15, C2 to C16, C5 to C2, C6 to C3, C7 to C4, C9 to C5, C11 to C6, C12 to C7, C13 to C8, C14 to C9, R4 to R1, R8 to R10, R5 to R2, R2 to R3, R9 to R4, R10 to R5, R1 to R6, R3 to R7, R6 to R8, R7 to R9, U2 to U1, U1 to U2
Other:
- note added: "Place close to pin 44"
- note added: "Place close to pin 45"
- note removed: "Place C6 close to pin 45"
- note removed: "Place C7 close to pin 44"

Commit message: Added files
Made changes to schematic to use unified daughter board S1 layout
Parts:
- removed J1: USB_C_Receptacle_USB2.0_16P, Connector_USB:USB_C_Receptacle_GCT_USB4105-xx-A_16P_TopMnt_Horizontal, symbol Connector:USB_C_Receptacle_USB2.0_16P
- removed R1, R2: 5.1kR, Resistor_SMD:R_01005_0402Metric, symbol Device:R
- added J1: 78171-0004, 122-LIB:PicoEZMate-Reinforced-Lite, symbol 122-LIB:PicoEZMate-Reinforced-Lite
- C1, C10, C11, C12, C13, C14, C15, C16, C2, C3, C4, C5, C6, C7, C8, C9: footprint Capacitor_SMD:C_01005_0402Metric -> Capacitor_SMD:C_0402_1005Metric
- R10, R3, R4, R5, R6, R7, R8, R9: footprint Resistor_SMD:R_01005_0402Metric -> Resistor_SMD:R_0402_1005Metric
Connections:
- net GND: now also J1.4 (Pin_4), J1.MP (MountPin)
- net USB_D+: now also J1.3 (Pin_3)
- net USB_D-: now also J1.2 (Pin_2)
- net VBUS: now also J1.1 (Pin_1)
- no-connect marks 4 -> 2
Other:
- note added: "Connector for cable to Unified Daughterboard S1 V1.1"
- note added: "LCSC: C588524"
- note removed: "LCSC: C5184243"

Commit message: Updated KiCad Files
Parts:
- C1, C10, C11, C12, C13, C14, C15, C16, C2, C3, C4, C5, C6, C7, C8, C9: footprint Capacitor_SMD:C_0402_1005Metric -> 122-LIB:C_0402_1005Metric-JLCSILK
- J2: symbol Connector_Generic:Conn_01x03 -> Connector_Generic_MountingPin:Conn_01x03_MountingPin; LCSC Part Number (none) -> C160403
- R1: renamed from R3; footprint Resistor_SMD:R_0402_1005Metric -> 122-LIB:R_0402_1005Metric-JLCSILK; now not fitted
- R2: renamed from R4; footprint Resistor_SMD:R_0402_1005Metric -> 122-LIB:R_0402_1005Metric-JLCSILK
- R3: renamed from R5; footprint Resistor_SMD:R_0402_1005Metric -> 122-LIB:R_0402_1005Metric-JLCSILK
- R4: renamed from R6; value 1k -> 1kR; footprint Resistor_SMD:R_0402_1005Metric -> 122-LIB:R_0402_1005Metric-JLCSILK
- R5: renamed from R7; value 1k -> 1kR; footprint Resistor_SMD:R_0402_1005Metric -> 122-LIB:R_0402_1005Metric-JLCSILK
- R6: renamed from R8; footprint Resistor_SMD:R_0402_1005Metric -> 122-LIB:R_0402_1005Metric-JLCSILK
- R7: renamed from R9; footprint Resistor_SMD:R_0402_1005Metric -> 122-LIB:R_0402_1005Metric-JLCSILK
- R8: renamed from R10; footprint Resistor_SMD:R_0402_1005Metric -> 122-LIB:R_0402_1005Metric-JLCSILK
- SW1, SW2: LCSC Part Number (none) -> C231329
- U1: LCSC Part Number (none) -> C26537
- U2: LCSC Part Number (none) -> C97521
- U3: LCSC Part Number (none) -> C2040; Manufacturer Part Number (none) -> RP2040; manufacturer Raspberry Pi -> (none)
- Y1: LCSC Part Number (none) -> C20625731
Connections:
- net GND: now also J2.MP (MountPin)
- net RUN: now also R8.2, U3.26 (RUN)
- net row0: now also U3.32 (GPIO21); no longer U3.38 (GPIO26_ADC0)
- net row1: now also U3.34 (GPIO22); no longer U3.39 (GPIO27_ADC1)
- net row2: now also U3.35 (GPIO23); no longer U3.37 (GPIO25)
- net row4: now also U3.37 (GPIO25); no longer U3.35 (GPIO23)
- net row5: now also U3.38 (GPIO26_ADC0); no longer U3.34 (GPIO22)
- net row6: now also U3.39 (GPIO27_ADC1); no longer U3.32 (GPIO21)
- net R_USB_D+: now reaches R2.1, U3.47 (USB_DP)
- net R_USB_D-: now reaches R3.1, U3.46 (USB_DM)
Other:
- moved on the sheet: C1, C2, R8, U1
