File: V2/switch-matrix.kicad_sch (KiCad schematic)
At the start: 256 parts

Commit message: Added updated files
Other:
- note added: "HOTSWAPS (LCSC): C41430893 DIODES (LCSC): C963381"
Changed lines of the file:
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@@
 	(generator_version "10.0")
 	(paper "D")
+	(text "HOTSWAPS (LCSC): C41430893\nDIODES (LCSC): C963381"
+		(exclude_from_sim no)
+		(at 12.954 14.732 0)
+		(effects
+			(font
+				(size 1.27 1.27)
+			)
+			(justify left)
+		)
+	)
 	(junction
 		(at 180.34 125.73)
