File: V2/kbplacer-preset/kbplacer-preset.kicad_pcb (KiCad board)
At the start: 2 copper layers, 2 parts

Commit message: Add files via upload
Parts:
- moved D_1 0.25 mm to (8.75, 10.3)
Routing:
- net Net-(D_1-A): track 11.8 -> 11.2 mm
Changed lines of the file:
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@@
 	(footprint "Diode_SMD:D_SOD-123"
 		(layer "B.Cu")
-		(at 8.5 10.3 90)
+		(at 8.75 10.3 90)
 		(descr "SOD-123")
 		(tags "SOD-123")
@@
 	)
 	(segment
+		(start 5.93 -1.27)
+		(end 5.93 -0.312641)
+		(width 0.75)
+		(layer "B.Cu")
+		(net "Net-(D_1-A)")
+	)
+	(segment
 		(start 6.318 -1.27)
 		(end 5.93 -1.27)
@@
 	)
 	(segment
-		(start 8.5 8.65)
-		(end 8.667321 8.482679)
-		(width 0.75)
-		(layer "B.Cu")
-		(net "Net-(D_1-A)")
-	)
-	(segment
-		(start 8.66732 1.07932)
-		(end 6.318 -1.27)
+		(start 6.80868 1.80868)
+		(end 7.871321 2.871321)
 		(width 0.75)
 		(layer "B.Cu")
@@
 	)
 	(segment
-		(start 9.546 6.361359)
-		(end 9.546 3.200641)
+		(start 8.75 4.992641)
+		(end 8.75 8.65)
 		(width 0.75)
 		(layer "B.Cu")
@@
 	)
 	(arc
-		(start 8.667321 8.482679)
-		(mid 9.317639 7.509409)
-		(end 9.546 6.361359)
+		(start 7.871321 2.871321)
+		(mid 8.521639 3.844591)
+		(end 8.75 4.992641)
 		(width 0.75)
 		(layer "B.Cu")
@@
 	)
 	(arc
-		(start 9.546 3.200641)
-		(mid 9.317638 2.05259)
-		(end 8.66732 1.07932)
+		(start 6.80868 1.80868)
+		(mid 6.158361 0.83541)
+		(end 5.93 -0.312641)
 		(width 0.75)
 		(layer "B.Cu")
@@
 		(polygon
 			(pts
-				(xy 8.6983 0.57997) (xy 8.474228 0.326844) (xy 8.352181 0.165638) (xy 8.231096 -0.011919) (xy 8.119986 -0.193383)
-				(xy 8.015802 -0.384731) (xy 7.929938 -0.564455) (xy 7.854357 -0.74855) (xy 7.797438 -0.914871) (xy 7.751975 -1.082004)
-				(xy 7.722342 -1.230796) (xy 7.704164 -1.378346) (xy 7.698508 -1.509381) (xy 7.703831 -1.638038)
-				(xy 7.705 -1.650766) (xy 6.123293 -1.464707) (xy 5.800233 -0.02) (xy 6.062522 -0.003676) (xy 6.353115 0.053344)
-				(xy 6.672127 0.15526) (xy 7.016139 0.305238) (xy 7.375519 0.502966) (xy 7.730336 0.740381) (xy 7.897669 0.869239)
-				(xy 8.046144 0.995355) (xy 8.16797 1.1103)
+				(xy 6.638994 0.971463) (xy 6.604431 0.792466) (xy 6.598132 0.678272) (xy 6.603115 0.556933) (xy 6.618284 0.451523)
+				(xy 6.645194 0.348541) (xy 6.677562 0.267507) (xy 6.720014 0.1926) (xy 6.765011 0.13492) (xy 6.818619 0.084467)
+				(xy 6.874656 0.046307) (xy 6.938533 0.015934) (xy 7.006816 -0.004861) (xy 7.082896 -0.017019) (xy 7.147761 -0.02)
+				(xy 5.280393 -1.079251) (xy 4.391962 -0.022593) (xy 4.53281 -0.010268) (xy 4.665542 0.011013) (xy 4.910985 0.079192)
+				(xy 5.131896 0.179752) (xy 5.331148 0.311912) (xy 5.510671 0.476077) (xy 5.671277 0.673358) (xy 5.812586 0.904678)
+				(xy 5.933091 1.169011) (xy 6.003953 1.370488)
 			)
 		)
@@
 		(polygon
 			(pts
-				(xy 8.843371 7.635149) (xy 8.760889 7.798253) (xy 8.695429 7.936953) (xy 8.615684 8.067236) (xy 8.568413 8.121209)
-				(xy 8.515121 8.163464) (xy 8.454992 8.190796) (xy 8.387209 8.2) (xy 8.592916 8.709564) (xy 9.1 8.754891)
-				(xy 9.084126 8.652704) (xy 9.105168 8.543218) (xy 9.167095 8.418279) (xy 9.280458 8.267368) (xy 9.35976 8.177018)
-				(xy 9.478413 8.034173)
-			)
-		)
+				(xy 8.375 7.75) (xy 8.395101 7.863825) (xy 8.416462 7.964548) (xy 8.421042 8.065398) (xy 8.4108 8.111764)
+				(xy 8.388876 8.153234) (xy 8.352774 8.188166) (xy 8.3 8.214918) (xy 8.75 8.651) (xy 9.2 8.214918)
+				(xy 9.156453 8.194277) (xy 9.123849 8.168213) (xy 9.086548 8.103669) (xy 9.077906 8.015718) (xy 9.104899 7.863825)
+				(xy 9.125 7.75)
+			)
+		)
